Commit message: feat: atualizando plug in

File: urdf/gazebo.xacro (robot description, xacro)
@@ -98,47 +98,40 @@
     </gazebo>
   </xacro:macro>
-  <xacro:macro
-    name="differential_controller"
+   <xacro:macro
+    name="skid_steer_controller"
     params="
       name
-      left_joint
-      right_joint
+      front_left_joint
+      front_right_joint
+      rear_left_joint
+      rear_right_joint
       wheel_diameter
       wheel_separation
+      publish_odom:=true
     "
   >
     <gazebo>
-      <plugin name="${name}_controller" filename="libgazebo_ros_diff_drive.so">
+      <plugin name="${name}_joint_states" filename="libgazebo_ros_joint_state_publisher.so">
+        <joint_name>${front_left_joint}</joint_name>
+        <joint_name>${front_right_joint}</joint_name>
+        <joint_name>${rear_left_joint}</joint_name>
+        <joint_name>${rear_right_joint}</joint_name>
+      </plugin>
+      <plugin name="${name}_controller" filename="libgazebo_ros_skid_steer_drive.so">
         <update_rate>50</update_rate>
-        <left_joint>${left_joint}</left_joint>
-        <right_joint>${right_joint}</right_joint>
+        <left_front_joint>${front_left_joint}</left_front_joint>
+        <right_front_joint>${front_right_joint}</right_front_joint>
+        <left_rear_joint>${rear_left_joint}</left_rear_joint>
+        <right_rear_joint>${rear_right_joint}</right_rear_joint>
         <wheel_diameter>${wheel_diameter}</wheel_diameter>
         <wheel_separation>${wheel_separation}</wheel_separation>
         <max_wheel_torque>20</max_wheel_torque>
         <max_wheel_acceleration>1.0</max_wheel_acceleration>
-        <command_topic>cmd_vel</command_topic>
-        <odometry_topic>odom</odometry_topic>
         <odometry_frame>odom</odometry_frame>
         <robot_base_frame>base_link</robot_base_frame>
-        <publish_odom>true</publish_odom>
-        <publish_odom_tf>true</publish_odom_tf>
-        <publish_wheel_tf>true</publish_wheel_tf>
-        <publish_wheel_joint_state>true</publish_wheel_joint_state>
+        <publish_odom>${publish_odom}</publish_odom>
+        <publish_odom_tf>${publish_odom}</publish_odom_tf>
       </plugin>
     </gazebo>
   </xacro:macro>
-  <!-- See: http://sdformat.org/tutorials?tut=sdformat_urdf_extensions&cat=specification -->
-  <xacro:macro
-    name="remove_friction"
-    params="position"
-  >
-    <gazebo reference="wheel_${position}_left">
-      <mu1>0.0</mu1>
-      <mu2>0.0</mu2>
-    </gazebo>
-    <gazebo reference="wheel_${position}_right">
-      <mu1>0.0</mu1>
-      <mu2>0.0</mu2>
-    </gazebo>
-  </xacro:macro>
 </robot>

Commit message: Revert "feat: atualizando plug in"
This reverts commit ca94ca284397a3381509c97399b6c20b32d88a46.

File: urdf/gazebo.xacro (robot description, xacro)
@@ -98,40 +98,47 @@
     </gazebo>
   </xacro:macro>
-   <xacro:macro
-    name="skid_steer_controller"
+  <xacro:macro
+    name="differential_controller"
     params="
       name
-      front_left_joint
-      front_right_joint
-      rear_left_joint
-      rear_right_joint
+      left_joint
+      right_joint
       wheel_diameter
       wheel_separation
-      publish_odom:=true
     "
   >
     <gazebo>
-      <plugin name="${name}_joint_states" filename="libgazebo_ros_joint_state_publisher.so">
-        <joint_name>${front_left_joint}</joint_name>
-        <joint_name>${front_right_joint}</joint_name>
-        <joint_name>${rear_left_joint}</joint_name>
-        <joint_name>${rear_right_joint}</joint_name>
-      </plugin>
-      <plugin name="${name}_controller" filename="libgazebo_ros_skid_steer_drive.so">
+      <plugin name="${name}_controller" filename="libgazebo_ros_diff_drive.so">
         <update_rate>50</update_rate>
-        <left_front_joint>${front_left_joint}</left_front_joint>
-        <right_front_joint>${front_right_joint}</right_front_joint>
-        <left_rear_joint>${rear_left_joint}</left_rear_joint>
-        <right_rear_joint>${rear_right_joint}</right_rear_joint>
+        <left_joint>${left_joint}</left_joint>
+        <right_joint>${right_joint}</right_joint>
         <wheel_diameter>${wheel_diameter}</wheel_diameter>
         <wheel_separation>${wheel_separation}</wheel_separation>
         <max_wheel_torque>20</max_wheel_torque>
         <max_wheel_acceleration>1.0</max_wheel_acceleration>
+        <command_topic>cmd_vel</command_topic>
+        <odometry_topic>odom</odometry_topic>
         <odometry_frame>odom</odometry_frame>
         <robot_base_frame>base_link</robot_base_frame>
-        <publish_odom>${publish_odom}</publish_odom>
-        <publish_odom_tf>${publish_odom}</publish_odom_tf>
+        <publish_odom>true</publish_odom>
+        <publish_odom_tf>true</publish_odom_tf>
+        <publish_wheel_tf>true</publish_wheel_tf>
+        <publish_wheel_joint_state>true</publish_wheel_joint_state>
       </plugin>
     </gazebo>
   </xacro:macro>
+  <!-- See: http://sdformat.org/tutorials?tut=sdformat_urdf_extensions&cat=specification -->
+  <xacro:macro
+    name="remove_friction"
+    params="position"
+  >
+    <gazebo reference="wheel_${position}_left">
+      <mu1>0.0</mu1>
+      <mu2>0.0</mu2>
+    </gazebo>
+    <gazebo reference="wheel_${position}_right">
+      <mu1>0.0</mu1>
+      <mu2>0.0</mu2>
+    </gazebo>
+  </xacro:macro>
 </robot>

Commit message: feat: retornando plug in

File: urdf/gazebo.xacro (robot description, xacro)
@@ -98,5 +98,5 @@
     </gazebo>
   </xacro:macro>
-  <xacro:macro
+   <xacro:macro
     name="differential_controller"
     params="
@@ -106,7 +106,12 @@
       wheel_diameter
       wheel_separation
+      publish_odom:=false
     "
   >
     <gazebo>
+      <plugin name="${name}_joint_states" filename="libgazebo_ros_joint_state_publisher.so">
+        <joint_name>${right_joint}</joint_name>
+        <joint_name>${left_joint}</joint_name>
+      </plugin>
       <plugin name="${name}_controller" filename="libgazebo_ros_diff_drive.so">
         <update_rate>50</update_rate>
@@ -117,12 +122,8 @@
         <max_wheel_torque>20</max_wheel_torque>
         <max_wheel_acceleration>1.0</max_wheel_acceleration>
-        <command_topic>cmd_vel</command_topic>
-        <odometry_topic>odom</odometry_topic>
         <odometry_frame>odom</odometry_frame>
         <robot_base_frame>base_link</robot_base_frame>
-        <publish_odom>true</publish_odom>
-        <publish_odom_tf>true</publish_odom_tf>
-        <publish_wheel_tf>true</publish_wheel_tf>
-        <publish_wheel_joint_state>true</publish_wheel_joint_state>
+        <publish_odom>${publish_odom}</publish_odom>
+        <publish_odom_tf>${publish_odom}</publish_odom_tf>
       </plugin>
     </gazebo>

Commit message: feat: adequando o diff drive ao skid steer

File: urdf/gazebo.xacro (robot description, xacro)
@@ -98,12 +98,17 @@
     </gazebo>
   </xacro:macro>
+<!-- Macro of skid steer using diff drive plugin as a coleague sugested-->
    <xacro:macro
-    name="differential_controller"
+    name="skid_steer_controller"
     params="
       name
-      left_joint
-      right_joint
-      wheel_diameter
-      wheel_separation
+      front_left_joint
+      front_right_joint
+      rear_left_joint
+      rear_right_joint
+      front_wheel_separation
+      rear_wheel_separation
+      front_wheel_diameter
+      rear_wheel_diameter
       publish_odom:=false
     "
@@ -111,13 +116,30 @@
     <gazebo>
       <plugin name="${name}_joint_states" filename="libgazebo_ros_joint_state_publisher.so">
-        <joint_name>${right_joint}</joint_name>
-        <joint_name>${left_joint}</joint_name>
+        <ros>
+          <remapping>~/out:=joint_states</remapping>
+        </ros>
+        <update_rate>50</update_rate>
+        <joint_names>
+          <joint_name>${front_right_joint}</joint_name>
+          <joint_name>${front_left_joint}</joint_name>
+          <joint_name>${rear_right_joint}</joint_name>
+          <joint_name>${rear_left_joint}</joint_name>
+        </joint_names>
       </plugin>
       <plugin name="${name}_controller" filename="libgazebo_ros_diff_drive.so">
+        <ros>
+          <command_topic>cmd_vel</command_topic>
+          <odometry_topic>odom</odometry_topic>
+        </ros>
         <update_rate>50</update_rate>
-        <left_joint>${left_joint}</left_joint>
-        <right_joint>${right_joint}</right_joint>
-        <wheel_diameter>${wheel_diameter}</wheel_diameter>
-        <wheel_separation>${wheel_separation}</wheel_separation>
+        <num_wheel_pairs>2</num_wheel_pairs>
+        <left_joint>${front_left_joint}</left_joint>
+        <right_joint>${front_right_joint}</right_joint>
+        <wheel_separation>${front_wheel_separation}</wheel_separation>
+        <wheel_diameter>${front_wheel_diameter}</wheel_diameter>
+        <left_joint>${rear_left_joint}</left_joint>
+        <right_joint>${rear_right_joint}</right_joint>
+        <wheel_separation>${rear_wheel_separation}</wheel_separation>
+        <wheel_diameter>${rear_wheel_diameter}</wheel_diameter>
         <max_wheel_torque>20</max_wheel_torque>
         <max_wheel_acceleration>1.0</max_wheel_acceleration>
@@ -126,20 +148,7 @@
         <publish_odom>${publish_odom}</publish_odom>
         <publish_odom_tf>${publish_odom}</publish_odom_tf>
+        <publish_wheel_tf>true</publish_wheel_tf>
       </plugin>
     </gazebo>
   </xacro:macro>
-  <!-- See: http://sdformat.org/tutorials?tut=sdformat_urdf_extensions&cat=specification -->
-  <xacro:macro
-    name="remove_friction"
-    params="position"
-  >
-    <gazebo reference="wheel_${position}_left">
-      <mu1>0.0</mu1>
-      <mu2>0.0</mu2>
-    </gazebo>
-    <gazebo reference="wheel_${position}_right">
-      <mu1>0.0</mu1>
-      <mu2>0.0</mu2>
-    </gazebo>
-  </xacro:macro>
 </robot>

Commit message: feat: adicionando rviz2 para abrir ao abrir o gazebo

File: urdf/gazebo.xacro (robot description, xacro)
@@ -18,5 +18,5 @@
         <update_rate>30</update_rate>
         <camera name="${name}_intrinsics">
-<!--          <distortion>
+          <!--          <distortion>
             <k1>0.1</k1>
             <k2>0.2</k2>
@@ -98,6 +98,6 @@
     </gazebo>
   </xacro:macro>
-<!-- Macro of skid steer using diff drive plugin as a coleague sugested-->
-   <xacro:macro
+  <!-- Macro of skid steer using diff drive plugin as a coleague sugested-->
+  <xacro:macro
     name="skid_steer_controller"
     params="
@@ -120,10 +120,8 @@
         </ros>
         <update_rate>50</update_rate>
-        <joint_names>
-          <joint_name>${front_right_joint}</joint_name>
-          <joint_name>${front_left_joint}</joint_name>
-          <joint_name>${rear_right_joint}</joint_name>
-          <joint_name>${rear_left_joint}</joint_name>
-        </joint_names>
+        <joint_name>${front_right_joint}</joint_name>
+        <joint_name>${front_left_joint}</joint_name>
+        <joint_name>${rear_right_joint}</joint_name>
+        <joint_name>${rear_left_joint}</joint_name>
       </plugin>
       <plugin name="${name}_controller" filename="libgazebo_ros_diff_drive.so">
